Commit message: Move large assets to Git LFS

File: public/models/iss/ISS.urdf (robot description, URDF)
Before this commit: robot ISS_stationaryFromNasa, 1 links, 0 joints
Links:
- link Root: geometry visual mesh filename=meshes/meshes/AMS2_000.obj scale=1. 1. 1.; visual mesh filename=meshes/meshes/Cube_001.obj scale=1. 1. 1.

File: public/models/iss/SD_SpaceStation_Ver05.urdf (robot description, URDF)
Before this commit: robot space_station, 1 links, 0 joints
Links:
- link Root: geometry collision mesh filename=meshes/SD_SpaceStation_Ver05.dae scale=100 100 100; visual mesh filename=meshes/SD_SpaceStation_Ver05.dae scale=100 100 100

Commit message: Improved UI

File: public/models/iss/ISS.urdf (robot description, URDF)
Before this commit: robot ISS_stationaryFromNasa, 1 links, 0 joints
Links:
- link Root: geometry visual mesh filename=meshes/AMS2_000.obj scale=1. 1. 1.; visual mesh filename=meshes/Cube_001.obj scale=1. 1. 1.
